File: smd-5v-3v3-usbmicro-powersupply-breakout/smd_5v_3v3_usbmicro_powersupply_breakout.kicad_pcb (KiCad board)
At the start: 2 copper layers, 32 x 48 mm, 12 parts, among them J1 USB_B_Micro, J2 THT 5V Jumper, J3 THT 3V3 Jumper, J4 SMD 5V Pad, J5 SMD 3V3 Pad, U1 LMS1585AIS-3.3

Commit message: Update usb micro psu (v04)
- Added a GND SMD pad
- Updated readme, schematic and 3d renders
Parts:
- added J6: SMD GND Pad, Connector_Wire:SolderWirePad_1x01_SMD_5x10mm, F.Cu at (160.0, 98.0)
Other:
- board text added: "5V & 3V3 USB Micro Power Supply Breakout Board v04"
- board text removed: "5V & 3V3 USB Micro Power Supply Breakout Board v03"
Changed lines of the file:
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@@
 		(title "5V & 3V3 USB Micro Power Supply Breakout Board")
 		(date "2025-02-11")
-		(rev "v03")
+		(rev "v04")
 	)
 	(layers
@@
 		)
 	)
+	(footprint "Connector_Wire:SolderWirePad_1x01_SMD_5x10mm"
+		(layer "F.Cu")
+		(at 160 98)
+		(descr "Wire Pad, Square, SMD Pad,  5mm x 10mm,")
+		(tags "MesurementPoint Square SMDPad 5mmx10mm ")
+		(property "Reference" "J6"
+			(at 4 2.5 0)
+			(layer "F.SilkS")
+			(effects
+				(font
+					(size 1 1)
+					(thickness 0.15)
+				)
+			)
+		)
+		(property "Value" "SMD GND Pad"
+			(at 0 6.35 0)
+			(layer "F.Fab")
+			(effects
+				(font
+					(size 1 1)
+					(thickness 0.15)
+				)
+			)
+		)
+		(property "Footprint" "Connector_Wire:SolderWirePad_1x01_SMD_5x10mm"
+			(at 0 0 0)
+			(unlocked yes)
+			(layer "F.Fab")
+			(hide yes)
+			(effects
+				(font
+					(size 1.27 1.27)
+					(thickness 0.15)
+				)
+			)
+		)
+		(property "Datasheet" ""
+			(at 0 0 0)
+			(unlocked yes)
+			(layer "F.Fab")
+			(hide yes)
+			(effects
+				(font
+					(size 1.27 1.27)
+					(thickness 0.15)
+				)
+			)
+		)
+		(property "Description" "Generic connector, single row, 01x01, script generated (kicad-library-utils/schlib/autogen/connector/)"
+			(at 0 0 0)
+			(unlocked yes)
+			(layer "F.Fab")
+			(hide yes)
+			(effects
+				(font
+					(size 1.27 1.27)
+					(thickness 0.15)
+				)
+			)
+		)
+		(property ki_fp_filters "Connector*:*_1x??_*")
+		(sheetname "Root")
+		(sheetfile "smd_5v_3v3_usbmicro_powersupply_breakout.kicad_sch")
+		(attr smd exclude_from_pos_files exclude_from_bom)
+		(fp_line
+			(start -2.75 -5.25)
+			(end -2.75 5.25)
+			(stroke
+				(width 0.05)
+				(type solid)
+			)
+			(layer "F.CrtYd")
+		)
+		(fp_line
+			(start -2.75 5.25)
+			(end 2.75 5.25)
+			(stroke
+				(width 0.05)
+				(type solid)
+			)
+			(layer "F.CrtYd")
+		)
+		(fp_line
+			(start 2.75 -5.25)
+			(end -2.75 -5.25)
+			(stroke
+				(width 0.05)
+				(type solid)
+			)
+			(layer "F.CrtYd")
+		)
+		(fp_line
+			(start 2.75 5.25)
+			(end 2.75 -5.25)
+			(stroke
+				(width 0.05)
+				(type solid)
+			)
+			(layer "F.CrtYd")
+		)
+		(fp_text user "${REFERENCE}"
+			(at 0 0 0)
+			(layer "F.Fab")
+			(effects
+				(font
+					(size 1 1)
+					(thickness 0.15)
+				)
+			)
+		)
+		(pad "1" smd rect
+			(at 0 0)
+			(size 5 10)
+			(layers "F.Cu" "F.Paste" "F.Mask")
+			(net 2 "GND")
+			(pinfunction "Pin_1")
+			(pintype "passive")
+		)
+	)
 	(footprint "Capacitor_SMD:CP_Elec_4x4.5"
 		(layer "F.Cu")
@@
 	)
 	(gr_text "5V"
-		(at 152.625 104 0)
+		(at 152.625 109.25 0)
 		(layer "F.SilkS")
 		(effects
@@
 		)
 	)
-	(gr_text "5V & 3V3\nUSB Micro\nPower Supply\nBreakout\nBoard v03"
+	(gr_text "5V & 3V3\nUSB Micro\nPower Supply\nBreakout\nBoard v04"
 		(at 165.25 138.25 0)
 		(layer "F.SilkS")
@@
 		)
 	)
+	(gr_text "GND"
+		(at 163 102.5 0)
+		(layer "F.SilkS")
+		(effects
+			(font
+				(size 1 1)
+				(thickness 0.15)
+			)
+			(justify left bottom)
+		)
+	)
 	(gr_text "3V3"
 		(at 175.25 108.5 0)
@@
 	)
 	(gr_text "GND"
-		(at 155.025 104 0)
+		(at 155.025 109.25 0)
 		(layer "F.SilkS")
 		(effects

Commit message: Kicad v9 pcb update (smd 5v/3v3 psu)
- Also corrected TVS diode part name
Parts:
- D1: value ESDB5V0WT -> PESD5V0X1UAB
